File: circuitry/low_pass/low_pass.kicad_sch (KiCad schematic)
At the start: 15 parts, among them U1 MCP6002-xP, U2 MCP6002-xP

Commit message: cleaner repo
Connections:
- net lowpass_gained is gone; now on net lowpass: C3.1, U1.1, U1.2 (-)
- net lowpass: no longer C1.1, R3.1, U2.1
- new net lowpass gained: C1.1, R3.1, U2.1
Other:
- moved on the sheet: C3, C4, R5, R6, U1C, V3
